File: cad/clintelli-board/clintelli-board.sch (KiCad schematic (older format))
At the start: 26 parts, among them J1 AudioJack4_Ground, J2 AudioJack3_Ground, J3 AudioJack3_Ground, P1 CONN_01X01, P2 CONN_01X01, P3 CONN_01X01, P4 CONN_01X01, SW1 SW_PUSH, U1 VDD, U2 ESP32-WROOM-32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

Commit message: clintelli board datasheets
Parts:
- gave numbers to parts that had none: 2
Changed lines of the file:
@@
 	3300 1600 3300 1750
 $Comp
-L power:VDD #PWR?
+L power:VDD #PWR0103
 U 1 1 5D519F04
 P 3300 1600
-F 0 "#PWR?" H 3300 1450 50  0001 C CNN
+F 0 "#PWR0103" H 3300 1450 50  0001 C CNN
 F 1 "VDD" H 3317 1773 50  0000 C CNN
 F 2 "" H 3300 1600 50  0001 C CNN
@@
 $EndComp
 $Comp
-L MCU_ST_STM32F3:STM32F302RETx U?
+L MCU_ST_STM32F3:STM32F302RETx U5
 U 1 1 5D4D89F4
 P 3400 3700
-F 0 "U?" H 3400 1811 50  0001 C CNN
+F 0 "U5" H 3400 1811 50  0001 C CNN
 F 1 "STM32F302RETx" H 3006 1720 50  0000 C CNN
 F 2 "Package_QFP:LQFP-64_10x10mm_P0.5mm" H 2800 2000 50  0001 R CNN
@@
 	3400 5600 3400 5750
 $Comp
-L clintelli-board-rescue:GND #PWR?
+L clintelli-board-rescue:GND #PWR0105
 U 1 1 5D54A877
 P 3400 5750
-F 0 "#PWR?" H 3400 5500 50  0001 C CNN
+F 0 "#PWR0105" H 3400 5500 50  0001 C CNN
 F 1 "GND" H 3405 5577 50  0000 C CNN
 F 2 "" H 3400 5750 50  0001 C CNN
@@
 	10050 4350 10050 4450
 $Comp
-L clintelli-board-rescue:GND #PWR?
+L clintelli-board-rescue:GND #PWR0106
 U 1 1 5D563A40
 P 10050 4450
-F 0 "#PWR?" H 10050 4200 50  0001 C CNN
+F 0 "#PWR0106" H 10050 4200 50  0001 C CNN
 F 1 "GND" H 10055 4277 50  0000 C CNN
 F 2 "" H 10050 4450 50  0001 C CNN
@@
 $EndComp
 $Comp
-L power:VDD #PWR?
+L power:VDD #PWR0107
 U 1 1 5D5A5FD7
 P 6500 7800
-F 0 "#PWR?" H 6500 7650 50  0001 C CNN
+F 0 "#PWR0107" H 6500 7650 50  0001 C CNN
 F 1 "VDD" H 6517 7973 50  0000 C CNN
 F 2 "" H 6500 7800 50  0001 C CNN
@@
 	4300 1750 4450 1750
 $Comp
-L power:VDD #PWR?
+L power:VDD #PWR0108
 U 1 1 5D5D7251
 P 4450 1750
-F 0 "#PWR?" H 4450 1600 50  0001 C CNN
+F 0 "#PWR0108" H 4450 1600 50  0001 C CNN
 F 1 "VDD" H 4467 1923 50  0000 C CNN
 F 2 "" H 4450 1750 50  0001 C CNN
@@
 $EndComp
 $Comp
-L clintelli-board-rescue:GND #PWR?
+L clintelli-board-rescue:GND #PWR0109
 U 1 1 5D641F68
 P 4550 9800
-F 0 "#PWR?" H 4550 9550 50  0001 C CNN
+F 0 "#PWR0109" H 4550 9550 50  0001 C CNN
 F 1 "GND" H 4550 9650 50  0000 C CNN
 F 2 "" H 4550 9800 60  0000 C CNN
@@
 I2C_SDA
 $Comp
-L power:VDD #PWR?
+L power:VDD #PWR0110
 U 1 1 5D81F5EC
 P 6850 1550
-F 0 "#PWR?" H 6850 1400 50  0001 C CNN
+F 0 "#PWR0110" H 6850 1400 50  0001 C CNN
 F 1 "VDD" H 6867 1723 50  0000 C CNN
 F 2 "" H 6850 1550 50  0001 C CNN
@@
 	13400 1850 13400 1800
 $Comp
-L power:VDDA #PWR?
+L power:VDDA #PWR0111
 U 1 1 5D8458E7
 P 3700 1600
-F 0 "#PWR?" H 3700 1450 50  0001 C CNN
+F 0 "#PWR0111" H 3700 1450 50  0001 C CNN
 F 1 "VDDA" H 3717 1773 50  0000 C CNN
 F 2 "" H 3700 1600 50  0001 C CNN
@@
 	3700 1750 3700 1900
 $Comp
-L power:VDDA #PWR?
+L power:VDDA #PWR0112
 U 1 1 5D849017
 P 13400 1750
-F 0 "#PWR?" H 13400 1600 50  0001 C CNN
+F 0 "#PWR0112" H 13400 1600 50  0001 C CNN
 F 1 "VDDA" H 13417 1923 50  0000 C CNN
 F 2 "" H 13400 1750 50  0001 C CNN
@@
 	13800 1850 13800 1750
 $Comp
-L power:VDD #PWR?
+L power:VDD #PWR0113
 U 1 1 5D84D116
 P 13800 1750
-F 0 "#PWR?" H 13800 1600 50  0001 C CNN
+F 0 "#PWR0113" H 13800 1600 50  0001 C CNN
 F 1 "VDD" H 13817 1923 50  0000 C CNN
 F 2 "" H 13800 1750 50  0001 C CNN
@@
 	13600 5300 13800 5300
 $Comp
-L clintelli-board-rescue:GND #PWR?
+L clintelli-board-rescue:GND #PWR0114
 U 1 1 5D855B76
 P 13600 5300
-F 0 "#PWR?" H 13600 5050 50  0001 C CNN
+F 0 "#PWR0114" H 13600 5050 50  0001 C CNN
 F 1 "GND" H 13605 5127 50  0000 C CNN
 F 2 "" H 13600 5300 50  0001 C CNN
@@
 Connection ~ 13500 6800
 $Comp
-L clintelli-board-rescue:R R?
+L clintelli-board-rescue:R R1
 U 1 1 5D3B5D43
 P 13950 6550
-F 0 "R?" H 14020 6596 50  0000 L CNN
+F 0 "R1" H 14020 6596 50  0000 L CNN
 F 1 "1M" H 14020 6505 50  0000 L CNN
 F 2 "" V 13880 6550 50  0001 C CNN
@@
 C6
 $Comp
-L clintelli-board-rescue:GND #PWR?
+L clintelli-board-rescue:GND #PWR0115
 U 1 1 5D469CCB
 P 12800 8400
-F 0 "#PWR?" H 12800 8150 50  0001 C CNN
+F 0 "#PWR0115" H 12800 8150 50  0001 C CNN
 F 1 "GND" H 12805 8227 50  0000 C CNN
 F 2 "" H 12800 8400 50  0001 C CNN
@@
 $EndComp
 $Comp
-L clintelli-board-rescue:GND #PWR?
+L clintelli-board-rescue:GND #PWR0116
 U 1 1 5D46A059
 P 14000 8400
-F 0 "#PWR?" H 14000 8150 50  0001 C CNN
+F 0 "#PWR0116" H 14000 8150 50  0001 C CNN
 F 1 "GND" H 14005 8227 50  0000 C CNN
 F 2 "" H 14000 8400 50  0001 C CNN
