File: cad/clintelli-board/clintelli-board.sch (KiCad schematic (older format))
At the start: 26 parts, among them J1 AudioJack4_Ground, J2 AudioJack3_Ground, J3 AudioJack3_Ground, P1 CONN_01X01, P2 CONN_01X01, P3 CONN_01X01, P4 CONN_01X01, SW1 SW_PUSH, U1 VDD, U2 ESP32-WROOM-32, U3 ADS1298xPAG, U4 ATECC608A-MAHDA, Y1 32MHz

Commit message: ESP32 wiring & 1st schematic export
Connections:
- net SPI3_SCK: now reaches U2.13 (IO14)
- net SPI3_SCK: now also U?.51 (PC10)
- net SPI3_MISO: now reaches U2.14 (IO12)
- net SPI3_MISO: now also U?.52 (PC11)
- net SPI3_MOSI: now reaches U2.16 (IO13)
- net SPI3_MOSI: now also U?.53 (PC12)
- net SPI3_NSS: now reaches U2.23 (IO15)
- net SPI3_NSS: now also U?.50 (PA15)
Changed lines of the file:
@@
 Text Notes 13200 7700 0    50   ~ 0
 Precordial Leads
+Wire Wire Line
+	4100 3600 4350 3600
+Wire Wire Line
+	2700 4800 2150 4800
+Wire Wire Line
+	2700 4900 2150 4900
+Wire Wire Line
+	2700 5000 2150 5000
+Text Label 4350 3600 0    50   ~ 0
+SPI3_NSS
+Text Label 2150 4800 0    50   ~ 0
+SPI3_SCK
+Text Label 2150 4900 0    50   ~ 0
+SPI3_MISO
+Text Label 2150 5000 0    50   ~ 0
+SPI3_MOSI
+Wire Wire Line
+	10650 2350 10900 2350
+Wire Wire Line
+	10650 2450 10900 2450
+Wire Wire Line
+	10650 2550 10900 2550
+Wire Wire Line
+	10650 2650 10900 2650
+Text Label 10900 2350 0    50   ~ 0
+SPI3_MISO
+Text Label 10900 2450 0    50   ~ 0
+SPI3_MOSI
+Text Label 10900 2550 0    50   ~ 0
+SPI3_SCK
+Text Label 10900 2650 0    50   ~ 0
+SPI3_NSS
 $EndSCHEMATC

Commit message: commit changes
Parts:
- removed R2: 1k, Capacitors_SMD:C_0805, symbol clintelli-board-rescue:R
- removed Y1: 32MHz, My Libraries:FA238-4pin_3.2x2.5mm_Offset, symbol clintelli-board-rescue:Crystal_GND24
- added R2: 1K, Resistor_SMD:R_0402_1005Metric, symbol Device:R
- added Y1: 32MHz, Crystal:Crystal_C38-LF_D3.0mm_L8.0mm_Horizontal_1EP_style2, symbol Device:Crystal_GND2
- C1: footprint (none) -> Capacitor_SMD:C_0805_2012Metric
- C3, C4, C5, C6, C7, C8, C9: footprint Capacitors_SMD:C_0805 -> Capacitor_SMD:C_0805_2012Metric
- D1: footprint LEDs:LED_0805 -> LED_SMD:LED_0805_2012Metric_Castellated
- J1: footprint (none) -> Connector_Audio:Jack_3.5mm_PJ320D_Horizontal; symbol Connector:AudioJack4_Ground -> Connector:AudioJack4
- J2, J3: footprint (none) -> Connector_Audio:Jack_3.5mm_CUI_SJ-3523-SMT_Horizontal; symbol Connector:AudioJack3_Ground -> Connector:AudioJack3
- L1: footprint (none) -> Inductor_SMD:L_6.3x6.3_H3
- P1, P2, P3, P4: footprint Mounting_Holes:MountingHole_2.2mm_M2_Pad -> MountingHole:MountingHole_2.2mm_M2_Pad
- R1: renamed from R?; footprint (none) -> Resistor_SMD:R_0402_1005Metric
- SW1: footprint My Libraries:SW_SPST_PTS830 -> Button_Switch_SMD:SW_Push_1P1T_NO_CK_KMR2; MFN CKN10589CT-ND -> (none)
- U1: footprint TO_SOT_Packages_SMD:SOT-23-5 -> Package_TO_SOT_SMD:SOT-23-5
- gave numbers to parts that had none: 1
Connections:
- net +3V3: now also R2.1
- net GND: now also Y1.2; no longer J1.G, J2.G, J3.G
- net OSC_IN: now also Y1.1
- net OSC_OUT: now also Y1.3
- net at D1.2 (A): now also R2.2
