File: cad/clintelli-board/_autosave-clintelli-board.sch (KiCad schematic (older format))
At the start: 26 parts, among them J1 AudioJack4_Ground, J2 AudioJack3_Ground, J3 AudioJack3_Ground, P1 CONN_01X01, P2 CONN_01X01, P3 CONN_01X01, P4 CONN_01X01, SW1 SW_PUSH, U1 VDD, U2 ESP32-WROOM-32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

Commit message: First PCB design attempt
Parts:
- SW1: footprint Button_Switch_THT:SW_PUSH_6mm -> Button_Switch_SMD:SW_Push_1P1T_NO_CK_KMR2
Changed lines of the file:
@@
 F 0 "SW1" V 4100 7650 50  0000 L CNN
 F 1 "SW_PUSH" V 4200 7550 50  0000 L CNN
-F 2 "Button_Switch_THT:SW_PUSH_6mm" H 4300 7450 60  0001 C CNN
+F 2 "Button_Switch_SMD:SW_Push_1P1T_NO_CK_KMR2" H 4300 7450 60  0001 C CNN
 F 3 "" H 4150 7900 60  0001 C CNN
 	1    4150 7900
