File: cad/clintelli-board/clintelli-board.kicad_pcb (KiCad board)
At the start: 2 copper layers, 26 parts, among them J1 AudioJack4_Ground, J2 AudioJack3_Ground, J3 AudioJack3_Ground, P1 CONN_01X01, P2 CONN_01X01, P3 CONN_01X01, P4 CONN_01X01, SW1 SW_PUSH, U1 VDD, U2 ESP32-WROOM-32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

Commit message: PCB layout second design attempt
Parts:
- moved P1 99.7 mm to (186.7, 133.3)
- moved P4 66.5 mm to (104.1, 88.9)
- moved C4 56.4 mm to (124.5, 134.6), turned to 270 degrees
- moved C6 46.8 mm to (146.1, 109.2), turned to 90 degrees
- moved C5 44.9 mm to (143.5, 135.9)
- moved L1 44.4 mm to (127.0, 128.3)
- moved Y1 44.0 mm to (139.1, 134.9), turned to 270 degrees
- moved C7 41.5 mm to (146.1, 105.4), turned to 90 degrees
- moved C9 38.9 mm to (151.1, 105.4), turned to 270 degrees
- moved U2 37.4 mm to (119.4, 110.5), turned to 90 degrees
- moved C3 36.9 mm to (157.8, 135.9), turned to 180 degrees
- moved C8 36.7 mm to (142.2, 105.4), turned to 180 degrees
- moved P3 31.5 mm to (185.4, 90.2)
- moved SW1 27.9 mm to (151.1, 135.9)
- moved R1 25.7 mm to (167.6, 132.1), turned to 270 degrees
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Routing:
- net GND: track 0.00 -> 39.6 mm, vias 0 -> 2
- net VDDA: track 29.8 -> 61.3 mm, vias 2 -> 0
- net /LL: track 10.3 -> 37.8 mm
- net /RA: track 18.3 -> 44.5 mm, vias 2 -> 0
- net /LA: track 23.4 -> 46.0 mm, vias 2 -> 0
- net /OSC_IN: track 34.0 -> 19.7 mm
- net /OSC_OUT: track 6.73 -> 20.4 mm
- net /SPI3_SCK: track 0.00 -> 12.9 mm, vias 0 -> 2
- net +3V3: track 47.4 -> 59.9 mm, vias 2 -> 0
- net VCC: track 3.52 -> 14.6 mm
- net /SPI1_SCK: track 2.27 -> 12.6 mm, vias 0 -> 2
- net /SPI1_MISO: track 6.43 -> 15.7 mm, vias 1 -> 2
- net /SPI3_MISO: track 0.00 -> 8.57 mm
- net /SPI1_MOSI: track 19.5 -> 11.1 mm, vias 2 -> 0
- net /SPI1_NSS: track 2.79 -> 11.0 mm
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- added copper zone on F.Cu, net GND
